Commit message: feat: fix typo, add udev script
Signed-off-by: Amadeusz Szymko <amadeuszszymko@gmail.com>

File: urdf/MTi_1.urdf (robot description, URDF)
Before this commit: robot mti_1, 1 links, 0 joints
Links:
- link imu_link: geometry visual mesh filename=package://bluespace_ai_xsens_mti_driver/urdf/MTi_1.stl scale=0.001 0.001 0.001

File: urdf/MTi_10.urdf (robot description, URDF)
Before this commit: robot mti_10, 1 links, 0 joints
Links:
- link imu_link: geometry visual mesh filename=package://bluespace_ai_xsens_mti_driver/urdf/MTi_10.stl scale=0.001 0.001 0.001

File: urdf/MTi_6xx.urdf (robot description, URDF)
Before this commit: robot mti_6xx, 1 links, 0 joints
Links:
- link imu_link: geometry visual mesh filename=package://bluespace_ai_xsens_mti_driver/urdf/MTi_6xx.stl scale=0.001 0.001 0.001
